Commit message: updating prius description to add lidar

File: prius_description/urdf/prius.urdf (robot description, URDF)
Before this commit: robot prius, 28 links, 27 joints
Links:
- added link vlp_16, mass 0.01; visual mesh filename=package://velodyne_description/meshes/VLP16_scan.dae
- link center_laser_link: mass 1 -> 0.83; geometry collision cylinder length=0.0717 radius=0.0516; visual mesh filename=package://velodyne_description/meshes/VLP16_base_1.dae
Joints:
- added joint vlp16_base_scan_joint: type fixed, parent center_laser_link, child vlp_16, origin xyz=0 0 0.0377 rpy=0 0 0
- joint center_laser_joint: origin xyz=0 0.4 1.8 rpy=0 0 -1.5707 -> xyz=0 0.4 1.5 rpy=0 0 -1.5707
